File: kicad/Adapterplatine/Adapterplatine.kicad_pcb (KiCad board)
At the start: 2 copper layers, 335 x 210 mm, 40 parts, among them J1 Conn_02x10_Top_Bottom, J10 Conn_01x04_Pin, J11 Conn_01x03_Pin, J12 Conn_01x02_Pin, J13 Conn_01x05_Pin, J14 Conn_01x02_Pin, J15 Conn_01x02_Pin, J16 Conn_01x05_Pin, J17 Conn_01x05_Pin, J18 Conn_01x05_Pin, J19 Conn_01x05_Pin, J2 DE9_Socket, J20 Conn_01x05_Pin, J21 Conn_01x05_Pin, J22 Conn_01x02_Pin, J23 Conn_01x02_Pin, J24 Conn_01x02_Pin, J25 Conn_01x02_Pin, J26 Conn_01x02_Pin, J27 Conn_01x05_Pin, J28 Conn_01x05_Pin, J29 Conn_01x02_Pin, J3 DE9_Pins, J30 Conn_01x05_Pin, J31 Conn_01x05_Pin, J32 Conn_01x05_Pin, J33 Conn_02x05_Top_Bottom, J34 Conn_01x02_Pin, J35 Conn_01x02_Pin, J4 DE9_Pins, J5 Conn_01x04_Pin, J6 Conn_01x04_Pin, J7 Conn_01x04_Pin, J8 Conn_01x04_Pin, J9 Conn_01x04_Pin

Commit message: Doku F421 Filamentsteuerung/ Doku Klipper Tabelle der Pins/ Code I2C Test/ Platinenanpassung KiCad/ printer.cfg Verbesserungen
Parts:
- added REF**: MountingHole_3.5mm_Pad, MountingHole:MountingHole_3.5mm_Pad, F.Cu at (283.0, 25.2)
- added REF**: MountingHole_3.5mm_Pad, MountingHole:MountingHole_3.5mm_Pad, F.Cu at (336.2, 202.5)
- added REF**: MountingHole_3.5mm_Pad, MountingHole:MountingHole_3.5mm_Pad, F.Cu at (289.5, 219.5)
- added REF**: MountingHole_3.5mm_Pad_Via, MountingHole:MountingHole_3.5mm_Pad_Via, F.Cu at (241.0, 53.8)
- added REF**: MountingHole_3.5mm_Pad_Via, MountingHole:MountingHole_3.5mm_Pad_Via, F.Cu at (334.5, 57.9)
- added REF**: MountingHole_3.5mm_Pad, MountingHole:MountingHole_3.5mm_Pad, F.Cu at (263.5, 54.0)
- added REF**: MountingHole_3.5mm_Pad, MountingHole:MountingHole_3.5mm_Pad, F.Cu at (297.2, 104.0)
- added REF**: MountingHole_3.5mm_Pad_Via, MountingHole:MountingHole_3.5mm_Pad_Via, F.Cu at (50.1, 53.6)
- added REF**: MountingHole_3.5mm_Pad_Via, MountingHole:MountingHole_3.5mm_Pad_Via, F.Cu at (50.1, 156.8)
- added REF**: MountingHole_3.5mm_Pad_Via, MountingHole:MountingHole_3.5mm_Pad_Via, F.Cu at (334.5, 115.8)
- added REF**: MountingHole_3.5mm_Pad, MountingHole:MountingHole_3.5mm_Pad, F.Cu at (32.0, 126.0)
- added REF**: MountingHole_3.5mm_Pad, MountingHole:MountingHole_3.5mm_Pad, F.Cu at (253.0, 142.0)
- added REF**: MountingHole_3.5mm_Pad, MountingHole:MountingHole_3.5mm_Pad, F.Cu at (236.0, 208.5)
- added REF**: MountingHole_3.5mm_Pad, MountingHole:MountingHole_3.5mm_Pad, F.Cu at (135.0, 112.5)
- added REF**: MountingHole_3.5mm_Pad, MountingHole:MountingHole_3.5mm_Pad, F.Cu at (126.0, 76.5)
- added REF**: MountingHole_3.5mm_Pad_Via, MountingHole:MountingHole_3.5mm_Pad_Via, F.Cu at (285.5, 115.9)
- added REF**: MountingHole_3.5mm_Pad_Via, MountingHole:MountingHole_3.5mm_Pad_Via, F.Cu at (241.0, 156.8)
- added REF**: MountingHole_3.5mm_Pad, MountingHole:MountingHole_3.5mm_Pad, F.Cu at (213.5, 53.5)
- added REF**: MountingHole_3.5mm_Pad_Via, MountingHole:MountingHole_3.5mm_Pad_Via, F.Cu at (285.5, 57.9)
- added REF**: MountingHole_3.5mm_Pad, MountingHole:MountingHole_3.5mm_Pad, F.Cu at (52.5, 213.5)
- added REF**: MountingHole_3.5mm_Pad, MountingHole:MountingHole_3.5mm_Pad, F.Cu at (330.2, 162.8)
- added REF**: MountingHole_3.5mm_Pad, MountingHole:MountingHole_3.5mm_Pad, F.Cu at (36.0, 26.0)
- added REF**: MountingHole_3.5mm_Pad, MountingHole:MountingHole_3.5mm_Pad, F.Cu at (325.8, 25.5)
- moved R1 42.0 mm to (214.0, 5.50)
- moved R2 42.0 mm to (224.2, 6.00)
- moved R3 42.0 mm to (231.7, 6.47)
- moved J9 36.2 mm to (177.9, 222.0)
- moved J35 35.2 mm to (35.8, 155.5)
- moved J34 28.3 mm to (35.8, 134.4)
- moved J8 25.9 mm to (136.8, 222.0)
- moved J10 25.7 mm to (216.4, 240.5)
- moved J11 25.7 mm to (186.4, 240.5)
- moved J13 25.7 mm to (198.9, 240.5)
- moved J18 25.2 mm to (177.0, 24.0)
- moved J31 23.0 mm to (56.4, 224.5)
- moved J32 21.1 mm to (70.4, 224.5)
- moved J20 20.5 mm to (191.4, 37.0)
- moved J19 20.2 mm to (190.9, 24.0)
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Other:
- board size 335 x 210 mm -> 333 x 210 mm

Commit message: Adapterplatine weitergeführt/ Doku F421
Parts:
- added FAN0: Conn_01x02_Pin, Connector_JST:JST_XH_B2B-XH-A_1x02_P2.50mm_Vertical, F.Cu at (142.0, 188.5)
- added FAN1: Conn_01x02_Pin, Connector_JST:JST_XH_B2B-XH-A_1x02_P2.50mm_Vertical, F.Cu at (151.5, 188.5)
- added FAN2: Conn_01x02_Pin, Connector_JST:JST_XH_B2B-XH-A_1x02_P2.50mm_Vertical, F.Cu at (161.5, 188.5)
- added I2C1: Conn_01x04_Pin, Connector_PinHeader_2.54mm:PinHeader_1x04_P2.54mm_Vertical, F.Cu at (269.3, 148.8)
- added Raspi_1: Conn_01x05_Pin, Connector_PinHeader_2.54mm:PinHeader_1x05_P2.54mm_Vertical, F.Cu at (269.3, 171.3)
- added Raspi_2: Conn_01x05_Pin, Connector_PinHeader_2.54mm:PinHeader_1x05_P2.54mm_Vertical, F.Cu at (294.0, 86.4)
- added X10__1: Conn_01x04_Pin, Connector_JST:JST_XH_B4B-XH-A_1x04_P2.50mm_Vertical, F.Cu at (210.5, 62.5)
- added X12__1: Conn_01x03_Pin, Connector_JST:JST_XH_B3B-XH-A_1x03_P2.50mm_Vertical, F.Cu at (288.5, 111.5)
- added X13__1: Conn_01x03_Pin, Connector_JST:JST_XH_B3B-XH-A_1x03_P2.50mm_Vertical, F.Cu at (288.5, 124.5)
- added X15__1: Conn_01x03_Pin, Connector_JST:JST_XH_B3B-XH-A_1x03_P2.50mm_Vertical, F.Cu at (280.0, 111.5)
- added X1__1: Conn_01x02_Pin, Connector_Phoenix_MSTB:PhoenixContact_MSTBA_2,5_2-G_1x02_P5.00mm_Horizontal, F.Cu at (52.7, 106.5)
- added X37__1: Conn_01x03_Pin, Connector_JST:JST_XH_B3B-XH-A_1x03_P2.50mm_Vertical, F.Cu at (271.5, 111.5)
- added X38__1: Conn_01x02_Pin, Connector_JST:JST_XH_B2B-XH-A_1x02_P2.50mm_Vertical, F.Cu at (171.2, 188.5)
- added X39__1: Conn_01x03_Pin, Connector_JST:JST_XH_B3B-XH-A_1x03_P2.50mm_Vertical, F.Cu at (271.5, 124.5)
- added X3__1: Conn_01x02_Pin, Connector_Phoenix_MSTB:PhoenixContact_MSTBA_2,5_2-G_1x02_P5.00mm_Horizontal, F.Cu at (52.7, 126.0)
- added X44__g1: Conn_01x02_Pin, Connector_JST:JST_XH_B2B-XH-A_1x02_P2.50mm_Vertical, F.Cu at (191.8, 188.5)
- added X44__r1: Conn_01x02_Pin, Connector_JST:JST_XH_B2B-XH-A_1x02_P2.50mm_Vertical, F.Cu at (181.8, 188.5)
- added X44__y1: Conn_01x04_Pin, Connector_Molex:Molex_KK-254_AE-6410-04A_1x04_P2.54mm_Vertical, F.Cu at (200.0, 189.0)
- added X44_b1: Conn_01x04_Pin, Connector_Molex:Molex_KK-254_AE-6410-04A_1x04_P2.54mm_Vertical, F.Cu at (216.0, 189.0)
- added X46__1: Conn_02x05_Top_Bottom, Connector_IDC:IDC-Header_2x05_P2.54mm_Vertical, F.Cu at (203.9, 201.0)
- added X48__PT1000_1: Conn_01x02_Pin, Connector_JST:JST_XH_B2B-XH-A_1x02_P2.50mm_Vertical, F.Cu at (142.0, 197.5)
- added X48__PT1000_2: Conn_01x02_Pin, Connector_JST:JST_XH_B2B-XH-A_1x02_P2.50mm_Vertical, F.Cu at (161.5, 197.5)
- added X48__Servo1: Conn_01x03_Pin, Connector_JST:JST_XH_B3B-XH-A_1x03_P2.50mm_Vertical, F.Cu at (84.5, 188.5)
- added X5__1: Conn_01x04_Pin, Connector_JST:JST_VH_B4P-VH_1x04_P3.96mm_Vertical, F.Cu at (93.0, 61.0)
- added X6__1: Conn_01x04_Pin, Connector_JST:JST_VH_B4P-VH_1x04_P3.96mm_Vertical, F.Cu at (117.1, 61.0)
- added X7__1: Conn_01x04_Pin, Connector_JST:JST_VH_B4P-VH_1x04_P3.96mm_Vertical, F.Cu at (142.0, 61.0)
- added X9__1: Conn_01x04_Pin, Connector_JST:JST_XH_B4B-XH-A_1x04_P2.50mm_Vertical, F.Cu at (192.5, 62.5)
- added X_EndStop4: Conn_01x03_Pin, Connector_JST:JST_XH_B3B-XH-A_1x03_P2.50mm_Vertical, F.Cu at (280.0, 124.5)
- added X_EndStop5: Conn_01x03_Pin, Connector_JST:JST_XH_B3B-XH-A_1x03_P2.50mm_Vertical, F.Cu at (280.0, 137.5)
- added X_EndStop6: Conn_01x03_Pin, Connector_JST:JST_XH_B3B-XH-A_1x03_P2.50mm_Vertical, F.Cu at (271.5, 137.5)
- X46: renamed from J33; footprint Connector_PinHeader_2.54mm:PinHeader_2x05_P2.54mm_Vertical -> Connector_IDC:IDC-Header_2x05_P2.54mm_Vertical
- moved R_X12 120.8 mm to (204.5, 126.0), turned to -90 degrees
- moved R_X13 120.7 mm to (211.0, 126.0), turned to -90 degrees
- moved R_X15 120.3 mm to (217.5, 126.0), turned to -90 degrees
- moved X52 76.2 mm to (225.4, 30.5), turned to 90 degrees
- moved X36B1 71.4 mm to (204.7, 219.1)
- moved J3 57.5 mm to (162.7, 220.0)
- moved X7 44.7 mm to (133.3, 223.5)
- moved J2 40.2 mm to (161.4, 226.0)
- moved J4 35.1 mm to (164.0, 213.5)
- moved X6 31.0 mm to (105.8, 223.5)
- moved X36A1 30.0 mm to (228.5, 219.1)
- moved REF** 29.9 mm to (261.5, 75.5)
- moved REF** 29.9 mm to (70.6, 75.4)
- moved REF** 29.9 mm to (183.5, 140.5)
- moved REF** 29.9 mm to (261.5, 178.5)
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- renumbered J13 to J2, J10 to J3, J11 to J4, R1 to R_X12, R2 to R_X13, R3 to R_X15, J34 to X1, J6 to X10, J19 to X12, J20 to X13, J31 to X15, J21 to X16, J15 to X20, J12 to X22, J22 to X23, J29 to X25_1, J18 to X28_1, J32 to X29_1, J35 to X3, J16 to X30, J17 to X31, J3 to X36A1, J2 to X36B1, J25 to X37, J23 to X38, J24 to X39, J14 to X40, J28 to X43, J27 to X44, J4 to X45, J1 to X48, J7 to X5, J30 to X52, J26 to X56, J8 to X6, J9 to X7, J5 to X9
Connections:
- R_X12 pad 1: unconnected-(R1-Pad1) -> Net-(X12-Pin_1)
- R_X12 pad 2: unconnected-(R1-Pad2) -> Net-(X12__1-Pin_1)
- R_X13 pad 1: unconnected-(R2-Pad1) -> Net-(X13-Pin_1)
- R_X13 pad 2: unconnected-(R2-Pad2) -> Net-(X13__1-Pin_1)
- R_X15 pad 1: unconnected-(R3-Pad1) -> Net-(X15__1-Pin_1)
- R_X15 pad 2: unconnected-(R3-Pad2) -> Net-(X15-Pin_1)
- X1 pad 1: unconnected-(J34-Pin_1-Pad1) -> Net-(X1-Pin_1)
- X1 pad 2: unconnected-(J34-Pin_2-Pad2) -> GND
- X10 pad 1: unconnected-(J6-Pin_1-Pad1) -> Net-(X10-Pin_1)
- X10 pad 2: unconnected-(J6-Pin_2-Pad2) -> Net-(X10-Pin_2)
- X10 pad 3: unconnected-(J6-Pin_3-Pad3) -> Net-(X10-Pin_3)
- X10 pad 4: unconnected-(J6-Pin_4-Pad4) -> Net-(X10-Pin_4)
- X12 pad 1: unconnected-(J19-Pin_1-Pad1) -> Net-(X12-Pin_1)
- X12 pad 2: unconnected-(J19-Pin_2-Pad2) -> GND
- X12 pad 4: unconnected-(J19-Pin_4-Pad4) -> GND
- X12 pad 5: unconnected-(J19-Pin_5-Pad5) -> Net-(X12-Pin_5)
- X13 pad 1: unconnected-(J20-Pin_1-Pad1) -> Net-(X13-Pin_1)
- X13 pad 2: unconnected-(J20-Pin_2-Pad2) -> GND
- X13 pad 4: unconnected-(J20-Pin_4-Pad4) -> GND
- X13 pad 5: unconnected-(J20-Pin_5-Pad5) -> Net-(X13-Pin_5)
- X15 pad 1: unconnected-(J31-Pin_1-Pad1) -> Net-(X15-Pin_1)
- X15 pad 2: unconnected-(J31-Pin_2-Pad2) -> GND
- X15 pad 4: unconnected-(J31-Pin_4-Pad4) -> GND
- X15 pad 5: unconnected-(J31-Pin_5-Pad5) -> Net-(X15-Pin_5)
- X29_1 pad 1: unconnected-(J32-Pin_1-Pad1) -> GND
- X29_1 pad 2: unconnected-(J32-Pin_2-Pad2) -> Net-(I2C1-Pin_1)
- X29_1 pad 3: unconnected-(J32-Pin_3-Pad3) -> Net-(I2C1-Pin_3)
- X29_1 pad 4: unconnected-(J32-Pin_4-Pad4) -> Net-(I2C1-Pin_4)
- X29_1 pad 5: unconnected-(J32-Pin_5-Pad5) -> GND
- X3 pad 1: unconnected-(J35-Pin_1-Pad1) -> Net-(X3-Pin_1)
- X3 pad 2: unconnected-(J35-Pin_2-Pad2) -> GND
- X37 pad 1: unconnected-(J25-Pin_1-Pad1) -> Net-(X37-Pin_1)
- X37 pad 2: unconnected-(J25-Pin_2-Pad2) -> Net-(X37-Pin_2)
- X38 pad 1: unconnected-(J23-Pin_1-Pad1) -> Net-(X38-Pin_1)
- X38 pad 2: unconnected-(J23-Pin_2-Pad2) -> Net-(X38-Pin_2)
- X39 pad 1: unconnected-(J24-Pin_1-Pad1) -> Net-(X39-Pin_1)
- X39 pad 2: unconnected-(J24-Pin_2-Pad2) -> Net-(X39-Pin_2)
- X44 pad 1: unconnected-(J27-Pin_1-Pad1) -> Net-(X44-Pin_1)
- X44 pad 2: unconnected-(J27-Pin_2-Pad2) -> Net-(X44-Pin_2)
- X44 pad 3: unconnected-(J27-Pin_3-Pad3) -> Net-(X44-Pin_3)
- X44 pad 4: unconnected-(J27-Pin_4-Pad4) -> Net-(X44-Pin_4)
- X44 pad 5: unconnected-(J27-Pin_5-Pad5) -> Net-(X44-Pin_5)
- X46 pad 1: unconnected-(J33-Pin_1-Pad1) -> Net-(X46-Pin_1)
- X46 pad 10: unconnected-(J33-Pin_10-Pad10) -> Net-(X46-Pin_10)
- X46 pad 2: unconnected-(J33-Pin_2-Pad2) -> Net-(X46-Pin_2)
- X46 pad 3: unconnected-(J33-Pin_3-Pad3) -> Net-(X46-Pin_3)
- X46 pad 5: unconnected-(J33-Pin_5-Pad5) -> GND
- X46 pad 7: unconnected-(J33-Pin_7-Pad7) -> Net-(X46-Pin_7)
- X48 pad 1: unconnected-(J1-Pin_1-Pad1) -> /GND TOOL
- X48 pad 10: unconnected-(J1-Pin_10-Pad10) -> Net-(X48-Pin_10)
- X48 pad 11: unconnected-(J1-Pin_11-Pad11) -> /VIN Tool1
- X48 pad 12: unconnected-(J1-Pin_12-Pad12) -> /VIN Tool1
- X48 pad 13: unconnected-(J1-Pin_13-Pad13) -> Net-(X48-Pin_13)
- X48 pad 14: unconnected-(J1-Pin_14-Pad14) -> Net-(X48-Pin_14)
- X48 pad 15: unconnected-(J1-Pin_15-Pad15) -> /GND TOOL
- X48 pad 16: unconnected-(J1-Pin_16-Pad16) -> /GND TOOL
- X48 pad 17: unconnected-(J1-Pin_17-Pad17) -> /VIN Tool0
- X48 pad 18: unconnected-(J1-Pin_18-Pad18) -> /VIN Tool0
- X48 pad 19: unconnected-(J1-Pin_19-Pad19) -> Net-(X48-Pin_19)
- X48 pad 2: unconnected-(J1-Pin_2-Pad2) -> /GND TOOL
- X48 pad 20: unconnected-(J1-Pin_20-Pad20) -> Net-(X48-Pin_20)
- X48 pad 4: unconnected-(J1-Pin_4-Pad4) -> Net-(FAN1-Pin_1)
- X48 pad 6: unconnected-(J1-Pin_6-Pad6) -> Net-(FAN2-Pin_2)
- X48 pad 7: unconnected-(J1-Pin_7-Pad7) -> Net-(X48-Pin_7)
- X48 pad 8: unconnected-(J1-Pin_8-Pad8) -> /GND TOOL
- X48 pad 9: unconnected-(J1-Pin_9-Pad9) -> Net-(FAN1-Pin_2)
- X5 pad 1: unconnected-(J7-Pin_1-Pad1) -> Net-(X5-Pin_1)
- X5 pad 2: unconnected-(J7-Pin_2-Pad2) -> Net-(X5-Pin_2)
- X5 pad 3: unconnected-(J7-Pin_3-Pad3) -> Net-(X5-Pin_3)
- X5 pad 4: unconnected-(J7-Pin_4-Pad4) -> Net-(X5-Pin_4)
- X6 pad 1: unconnected-(J8-Pin_1-Pad1) -> Net-(X6-Pin_1)
- X6 pad 2: unconnected-(J8-Pin_2-Pad2) -> Net-(X6-Pin_2)
- X6 pad 3: unconnected-(J8-Pin_3-Pad3) -> Net-(X6-Pin_3)
- X6 pad 4: unconnected-(J8-Pin_4-Pad4) -> Net-(X6-Pin_4)
- X7 pad 1: unconnected-(J9-Pin_1-Pad1) -> Net-(X7-Pin_1)
- X7 pad 2: unconnected-(J9-Pin_2-Pad2) -> Net-(X7-Pin_2)
- X7 pad 3: unconnected-(J9-Pin_3-Pad3) -> Net-(X7-Pin_3)
- X7 pad 4: unconnected-(J9-Pin_4-Pad4) -> Net-(X7-Pin_4)
- X9 pad 1: unconnected-(J5-Pin_1-Pad1) -> Net-(X9-Pin_1)
- X9 pad 2: unconnected-(J5-Pin_2-Pad2) -> Net-(X9-Pin_2)
- X9 pad 3: unconnected-(J5-Pin_3-Pad3) -> Net-(X9-Pin_3)
- X9 pad 4: unconnected-(J5-Pin_4-Pad4) -> Net-(X9-Pin_4)
Routing:
- net Net-(X7-Pin_1): track 0.00 -> 2.76 mm
- net Net-(X6-Pin_4): track 0.00 -> 0.76 mm

Commit message: Doku F421/ Klipper ython modul erstellt/ KiCad Adapterplatine
Parts:
- added X48_Tool0: Conn_01x02_Pin, Connector_Phoenix_MSTB:PhoenixContact_MSTBA_2,5_2-G_1x02_P5.00mm_Horizontal, F.Cu at (104.5, 205.0)
- added X48_Tool1: Conn_01x02_Pin, Connector_Phoenix_MSTB:PhoenixContact_MSTBA_2,5_2-G_1x02_P5.00mm_Horizontal, F.Cu at (118.0, 205.0)

Commit message: Adapterplatinen Update
Parts:
- added MAX31865_IN1: Conn_01x08_Pin, Connector_PinSocket_2.54mm:PinSocket_1x08_P2.54mm_Vertical, F.Cu at (73.0, 64.2)
- added MAX31865_OUT1: Conn_01x04_Pin, Connector_PinSocket_2.54mm:PinSocket_1x04_P2.54mm_Vertical, F.Cu at (51.4, 59.1)
- added PowerOn1: Conn_01x02_Pin, Connector_PinHeader_2.54mm:PinHeader_1x02_P2.54mm_Vertical, F.Cu at (343.5, 99.5)
- added SPI4: Conn_02x04_Top_Bottom, Connector_PinHeader_2.54mm:PinHeader_2x04_P2.54mm_Vertical, F.Cu at (289.7, 157.5)
- added T_Bauraum1: Conn_01x02_Pin, Connector_JST:JST_XH_B2B-XH-A_1x02_P2.50mm_Vertical, F.Cu at (277.0, 172.0)
- added T_HeizE1: Conn_01x02_Pin, Connector_JST:JST_XH_B2B-XH-A_1x02_P2.50mm_Vertical, F.Cu at (277.0, 151.0)
- added T_Heizbett1: Conn_01x02_Pin, Connector_JST:JST_XH_B2B-XH-A_1x02_P2.50mm_Vertical, F.Cu at (277.0, 161.5)
- moved I2C1 13.7 mm to (283.0, 149.9)
- moved REF** 11.8 mm to (346.5, 32.6)
- moved REF** 11.8 mm to (346.5, 90.5)
- moved REF** 11.8 mm to (297.5, 90.6)
- moved REF** 11.8 mm to (297.5, 32.6)
- moved REF** 11.8 mm to (324.5, 59.0)
- moved Raspi_2 11.8 mm to (291.5, 74.9)
- renumbered X_EndStop6 to Not_Aus1
Connections:
- FAN0 pad 1: unconnected-(FAN0-Pin_1-Pad1) -> Net-(FAN0-Pin_1)
- FAN0 pad 2: unconnected-(FAN0-Pin_2-Pad2) -> Net-(FAN0-Pin_2)
- Not_Aus1 pad 2: unconnected-(X_EndStop6-Pin_2-Pad2) -> Net-(Not_Aus1-Pin_2)
- Not_Aus1 pad 3: unconnected-(X_EndStop6-Pin_3-Pad3) -> Net-(Not_Aus1-Pin_3)
- X16 pad 4: unconnected-(X16-Pin_4-Pad4) -> Net-(Not_Aus1-Pin_2)
- X16 pad 5: unconnected-(X16-Pin_5-Pad5) -> Net-(Not_Aus1-Pin_3)
- X20 pad 1: unconnected-(X20-Pin_1-Pad1) -> Net-(T_HeizE1-Pin_1)
- X20 pad 2: unconnected-(X20-Pin_2-Pad2) -> Net-(T_HeizE1-Pin_2)
- X22 pad 1: unconnected-(X22-Pin_1-Pad1) -> Net-(MAX31865_OUT1-Pin_2)
- X22 pad 2: unconnected-(X22-Pin_2-Pad2) -> Net-(MAX31865_OUT1-Pin_3)
- X23 pad 1: unconnected-(X23-Pin_1-Pad1) -> Net-(T_Bauraum1-Pin_1)
- X23 pad 2: unconnected-(X23-Pin_2-Pad2) -> Net-(T_Bauraum1-Pin_2)
- X25_1 pad 1: unconnected-(X25_1-Pin_1-Pad1) -> Net-(FAN0-Pin_1)
- X25_1 pad 2: unconnected-(X25_1-Pin_2-Pad2) -> Net-(FAN0-Pin_2)
- X29_1 pad 2: Net-(I2C1-Pin_1) -> unconnected-(X29_1-Pin_2-Pad2)
- X29_1 pad 3: Net-(I2C1-Pin_3) -> Net-(I2C1-Pin_4)
- X29_1 pad 4: Net-(I2C1-Pin_4) -> Net-(I2C1-Pin_3)
- X43 pad 1: unconnected-(X43-Pin_1-Pad1) -> GND
- X43 pad 2: unconnected-(X43-Pin_2-Pad2) -> Net-(PowerOn1-Pin_1)
- X43 pad 4: unconnected-(X43-Pin_4-Pad4) -> Net-(PowerOn1-Pin_2)
- X43 pad 5: unconnected-(X43-Pin_5-Pad5) -> Net-(I2C1-Pin_1)
- X56 pad 1: unconnected-(X56-Pin_1-Pad1) -> Net-(T_Heizbett1-Pin_1)
- X56 pad 2: unconnected-(X56-Pin_2-Pad2) -> Net-(T_Heizbett1-Pin_2)
Other:
- board size 333 x 210 mm -> 334.5 x 210 mm
