File: kicad/Adapterplatine/Adapterplatine.kicad_pcb (KiCad board)
At the start: 6 copper layers, 333 x 210 mm, 102 parts, among them J2 Conn_01x05_Pin, J3 Conn_01x04_Pin, J4 Conn_01x03_Pin, X1 Conn_01x02_Pin, X10 Conn_01x04_Pin, X12 Conn_01x05_Pin, X13 Conn_01x05_Pin, X15 Conn_01x05_Pin, X16 Conn_01x05_Pin, X20 Conn_01x02_Pin, X22 Conn_01x02_Pin, X23 Conn_01x02_Pin, X25_1 Conn_01x02_Pin, X28_1 Conn_01x05_Pin, X29_1 Conn_01x05_Pin, X3 Conn_01x02_Pin, X30 Conn_01x05_Pin, X31 Conn_01x05_Pin, X36A1 DE9_Pins, X36B1 DE9_Socket, X37 Conn_01x02_Pin, X38 Conn_01x02_Pin, X39 Conn_01x02_Pin, X40 Conn_01x02_Pin, X43 Conn_01x05_Pin, X44 Conn_01x05_Pin, X44__g1 Conn_01x02_Pin, X44__r1 Conn_01x04_Pin, X44__y1 Conn_01x02_Pin, X44_b1 Conn_01x04_Pin, X45 DE9_Pins, X46 Conn_02x05_Top_Bottom, X46__1 Conn_02x05_Top_Bottom, X48 Conn_02x10_Top_Bottom, X5 Conn_01x04_Pin, X52 Conn_01x05_Pin, X56 Conn_01x02_Pin, X6 Conn_01x04_Pin, X7 Conn_01x04_Pin, X9 Conn_01x04_Pin

Commit message: Umsortierung/ Erste Leitungung Adapterplatine
Parts:
- added J1: Conn_01x05, Connector_PinSocket_2.54mm:PinSocket_1x05_P2.54mm_Vertical, F.Cu at (315.9, 112.9)
- moved R3 10.2 mm to (39.6, 218.3)
Routing:
- net Net-(MAX31865_OUT1-Pin_2): track 0.00 -> 385.0 mm
- net Net-(MAX31865_OUT1-Pin_3): track 0.00 -> 384.6 mm
- net Net-(EndStopZ3-Pin_3): track 0.00 -> 343.4 mm
- net Net-(NTC_Headbed2-Pin_2): track 0.00 -> 276.7 mm
- net Net-(NTC_Headbed2-Pin_1): track 0.00 -> 273.6 mm
- net Net-(MotorExtruder5-Pin_4): track 0.00 -> 177.8 mm, vias 0 -> 1
- net Net-(MotorExtruder5-Pin_2): track 0.00 -> 171.9 mm
- net Net-(MotorY2-Pin_4): track 0.00 -> 170.7 mm, vias 0 -> 1
- net Net-(MotorExtruder5-Pin_3): track 0.00 -> 170.7 mm, vias 0 -> 1
- net Net-(MotorX1-Pin_2): track 0.00 -> 170.3 mm
- net Net-(MotorY2-Pin_3): track 0.76 -> 170.8 mm
- net Net-(MotorX1-Pin_4): track 0.00 -> 169.4 mm
- net Net-(MotorZ3-Pin_4): track 0.00 -> 169.1 mm
- net Net-(MotorY2-Pin_2): track 0.00 -> 168.9 mm
- net Net-(MotorZ3-Pin_2): track 0.00 -> 168.7 mm
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
Commit message: Leitungsverlegung Adapterplatine abgeschlossen
Parts:
- added R10: 10k, Resistor_THT:R_Axial_DIN0207_L6.3mm_D2.5mm_P10.16mm_Horizontal, F.Cu at (31.9, 40.0)
- added R11: 20k, Resistor_THT:R_Axial_DIN0207_L6.3mm_D2.5mm_P10.16mm_Horizontal, F.Cu at (45.1, 40.0)
- added R4: 10k, Resistor_THT:R_Axial_DIN0207_L6.3mm_D2.5mm_P10.16mm_Horizontal, F.Cu at (31.9, 55.0)
- added R5: 20k, Resistor_THT:R_Axial_DIN0207_L6.3mm_D2.5mm_P10.16mm_Horizontal, F.Cu at (45.0, 55.0)
- added R6: 10k, Resistor_THT:R_Axial_DIN0207_L6.3mm_D2.5mm_P10.16mm_Horizontal, F.Cu at (31.9, 50.0)
- added R7: 20k, Resistor_THT:R_Axial_DIN0207_L6.3mm_D2.5mm_P10.16mm_Horizontal, F.Cu at (44.9, 50.0)
- added R8: 10k, Resistor_THT:R_Axial_DIN0207_L6.3mm_D2.5mm_P10.16mm_Horizontal, F.Cu at (31.9, 45.0)
- added R9: 20k, Resistor_THT:R_Axial_DIN0207_L6.3mm_D2.5mm_P10.16mm_Horizontal, F.Cu at (45.1, 45.0)
- R1, R2, R3: footprint Resistor_THT:R_Axial_DIN0207_L6.3mm_D2.5mm_P2.54mm_Vertical -> Resistor_THT:R_Axial_DIN0207_L6.3mm_D2.5mm_P10.16mm_Horizontal
- X44__g1: value Conn_01x02_Pin -> Conn_01x04_Pin; footprint Connector_JST:JST_XH_B2B-XH-A_1x02_P2.50mm_Vertical -> Connector_Molex:Molex_KK-254_AE-6410-04A_1x04_P2.54mm_Vertical
- X44_b1: value Conn_01x04_Pin -> Conn_01x02_Pin; footprint Connector_Molex:Molex_KK-254_AE-6410-04A_1x04_P2.54mm_Vertical -> Connector_JST:JST_XH_B2B-XH-A_1x02_P2.50mm_Vertical
- moved X44_b1 34.2 mm to (180.8, 188.0)
- moved X25_1 22.4 mm to (265.3, 34.5)
- moved X43 22.0 mm to (261.4, 24.0)
- moved RP2040-PIN0-8 20.4 mm to (336.3, 125.6), turned to -90 degrees
- moved X52 18.4 mm to (243.4, 34.5)
- moved X44__g1 18.3 mm to (199.0, 188.5)
- moved X44 18.0 mm to (242.9, 24.0)
- moved R1 17.1 mm to (204.6, 49.0), turned to 180 degrees
- moved X44__r1 15.8 mm to (214.8, 188.6)
- moved X39 12.7 mm to (231.0, 24.0)
- moved X37 10.8 mm to (221.7, 34.5)
- moved R3 10.5 mm to (29.4, 220.5), turned to 0 degrees
- moved J1 10.2 mm to (315.9, 123.1), turned to 180 degrees
- moved X38 10.0 mm to (221.7, 24.0)
- moved R2 9.45 mm to (204.6, 42.5), turned to 180 degrees
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Connections:
- X30 pad 2: Net-(RP2040-PIN0-8-Pin_6) -> Net-(X30-Pin_2)
- X30 pad 3: Net-(RP2040-PIN0-8-Pin_5) -> Net-(X30-Pin_3)
- X31 pad 2: Net-(RP2040-PIN0-8-Pin_4) -> Net-(X31-Pin_2)
- X31 pad 3: Net-(RP2040-PIN0-8-Pin_3) -> Net-(X31-Pin_3)
- X44__g1 pad 1: Net-(X44-Pin_2) -> Net-(X44-Pin_4)
- X44__g1 pad 2: Net-(X44-Pin_4) -> unconnected-(X44__g1-Pin_2-Pad2)
- X44__r1 pad 3: unconnected-(X44__r1-Pin_3-Pad3) -> Net-(X44-Pin_2)
- X44__r1 pad 4: Net-(X44-Pin_2) -> unconnected-(X44__r1-Pin_4-Pad4)
- X44_b1 pad 1: Net-(X44-Pin_1) -> Net-(X44-Pin_2)
- X44_b1 pad 2: unconnected-(X44_b1-Pin_2-Pad2) -> Net-(X44-Pin_1)
Routing:
- net Net-(RP2040-PIN0-8-Pin_3): track 0.00 -> 322.7 mm
- net Net-(RP2040-PIN0-8-Pin_4): track 0.00 -> 321.2 mm
- net Net-(RP2040-PIN0-8-Pin_5): track 0.00 -> 320.2 mm
- net Net-(RP2040-PIN0-8-Pin_6): track 0.00 -> 319.1 mm
- net Net-(X46-Pin_3): track 0.00 -> 305.9 mm, vias 0 -> 1
- net Net-(X46-Pin_10): track 0.00 -> 305.2 mm
- net Net-(X46-Pin_2): track 0.00 -> 300.6 mm
- net Net-(X46-Pin_7): track 0.00 -> 299.7 mm, vias 0 -> 1
- net Net-(I2C1-Pin_3): track 0.00 -> 272.1 mm, vias 0 -> 1
- net Net-(I2C1-Pin_4): track 0.00 -> 271.6 mm, vias 0 -> 2
- net /Fan/X48-FAN0 PIN9: track 0.00 -> 242.9 mm
- net /Motor Driver/X48-Servo-PIN10: track 0.00 -> 239.9 mm, vias 0 -> 1
- net /Motor Driver/X48-Servo-PIN7: track 0.00 -> 230.9 mm
- net Net-(FAN0-Pin_2): track 0.00 -> 205.0 mm, vias 0 -> 1
- net Net-(FAN0-Pin_1): track 0.00 -> 204.9 mm, vias 0 -> 1
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