File: kicad/Adapterplatine/Adapterplatine.kicad_pcb (KiCad board)
At the start: 6 copper layers, 333 x 210 mm, 111 parts, among them J1 Conn_01x05, J2 Conn_01x05_Pin, J3 Conn_01x04_Pin, J4 Conn_01x03_Pin, X1 Conn_01x02_Pin, X10 Conn_01x04_Pin, X12 Conn_01x05_Pin, X13 Conn_01x05_Pin, X15 Conn_01x05_Pin, X16 Conn_01x05_Pin, X20 Conn_01x02_Pin, X22 Conn_01x02_Pin, X23 Conn_01x02_Pin, X25_1 Conn_01x02_Pin, X28_1 Conn_01x05_Pin, X29_1 Conn_01x05_Pin, X3 Conn_01x02_Pin, X30 Conn_01x05_Pin, X31 Conn_01x05_Pin, X36A1 DE9_Pins, X36B1 DE9_Socket, X37 Conn_01x02_Pin, X38 Conn_01x02_Pin, X39 Conn_01x02_Pin, X40 Conn_01x02_Pin, X43 Conn_01x05_Pin, X44 Conn_01x05_Pin, X44__g1 Conn_01x04_Pin, X44__r1 Conn_01x04_Pin, X44__y1 Conn_01x02_Pin, X44_b1 Conn_01x02_Pin, X45 DE9_Pins, X46 Conn_02x05_Top_Bottom, X46__1 Conn_02x05_Top_Bottom, X48 Conn_02x10_Top_Bottom, X5 Conn_01x04_Pin, X52 Conn_01x05_Pin, X56 Conn_01x02_Pin, X6 Conn_01x04_Pin, X7 Conn_01x04_Pin, X9 Conn_01x04_Pin

Commit message: Bessere Verlegungen Adapterplatine
Parts:
- removed X46__1: Conn_02x05_Top_Bottom, Connector_IDC:IDC-Header_2x05_P2.54mm_Vertical
- added 230V_Platine1: Conn_02x05_Odd_Even, Connector_IDC:IDC-Header_2x05_P2.54mm_Vertical, F.Cu at (202.8, 200.5)
- RP2040-PIN14-32: value Conn_01x05_Pin -> Conn_01x09_Pin
- SPI4: value Conn_02x04_Top_Bottom -> Conn_02x04_Odd_Even
- X46: value Conn_02x05_Top_Bottom -> Conn_02x05_Odd_Even
- moved R7 10.2 mm to (55.1, 50.0), turned to 180 degrees
- moved R11 10.2 mm to (55.2, 40.0), turned to 180 degrees
- moved R5 10.1 mm to (55.1, 55.0), turned to 180 degrees
- moved R9 9.92 mm to (55.0, 45.0), turned to 180 degrees
- moved SPI4 8.09 mm to (289.0, 149.4), turned to 0 degrees
- moved X46 0.06 mm to (30.9, 64.8)
Connections:
- Rasp1 pad 4: Net-(Rasp1-Pin_4) -> unconnected-(Rasp1-Pin_4-Pad4)
- SPI4 pad 1: GND -> +5V
- SPI4 pad 2: Net-(MAX31865_IN1-Pin_4) -> GND
- SPI4 pad 3: Net-(MAX31865_IN1-Pin_6) -> Net-(MAX31865_IN1-Pin_7)
- SPI4 pad 4: GND -> Net-(MAX31865_IN1-Pin_4)
- SPI4 pad 5: +5V -> Net-(MAX31865_IN1-Pin_5)
- SPI4 pad 6: Net-(MAX31865_IN1-Pin_7) -> Net-(MAX31865_IN1-Pin_6)
- SPI4 pad 7: Net-(MAX31865_IN1-Pin_5) -> /platines/+3.3V
- SPI4 pad 8: unconnected-(SPI4-Pin_8-Pad8) -> GND
- UART0 pad 4: Net-(Rasp1-Pin_4) -> unconnected-(UART0-Pin_4-Pad4)
- UART0 pad 5: Net-(RP2040-PIN14-32-Pin_9) -> unconnected-(UART0-Pin_5-Pad5)
- X29_1 pad 2: +3.3V -> /platines/+3.3V
- X46 pad 1: +5V -> Net-(230V_Platine1-Pin_10)
- X46 pad 10: Net-(X46-Pin_10) -> GND
- X46 pad 2: Net-(X46-Pin_2) -> +5V
- X46 pad 4: unconnected-(X46-Pin_4-Pad4) -> Net-(230V_Platine1-Pin_8)
- X46 pad 5: GND -> Net-(230V_Platine1-Pin_7)
- X46 pad 6: unconnected-(X46-Pin_6-Pad6) -> Net-(230V_Platine1-Pin_6)
- X46 pad 8: unconnected-(X46-Pin_8-Pad8) -> Net-(230V_Platine1-Pin_4)
- X46 pad 9: unconnected-(X46-Pin_9-Pad9) -> Net-(230V_Platine1-Pin_3)
Routing:
- net Net-(230V_Platine1-Pin_10): track 0.00 -> 322.1 mm
- net Net-(230V_Platine1-Pin_7): track 0.00 -> 313.4 mm
- net Net-(X46-Pin_10): track 305.2 -> 0.00 mm
- net Net-(230V_Platine1-Pin_8): track 0.00 -> 301.0 mm
- net Net-(X46-Pin_2): track 300.6 -> 0.00 mm
- net Net-(230V_Platine1-Pin_3): track 0.00 -> 299.5 mm
- net Net-(230V_Platine1-Pin_6): track 0.00 -> 297.4 mm
- net Net-(230V_Platine1-Pin_4): track 0.00 -> 293.8 mm
- net /platines/+3.3V: track 0.00 -> 289.0 mm, vias 0 -> 1
- net Net-(Rasp1-Pin_4): track 123.9 -> 0.00 mm
- net Net-(RP2040-PIN14-32-Pin_9): track 169.2 -> 56.7 mm
- net Net-(RP2040-PIN0-8-Pin_6): track 319.1 -> 342.9 mm
- net Net-(RP2040-PIN0-8-Pin_5): track 320.2 -> 341.3 mm
- net Net-(MAX31865_IN1-Pin_5): track 52.8 -> 73.5 mm, vias 1 -> 0
- net Net-(RP2040-PIN0-8-Pin_4): track 321.2 -> 339.8 mm
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- removed copper zone on In3.Cu, net +3.3V

Commit message: Aufnahme des i2C Splitters am Druckkopf/ Kleine Änderungen Platine
Parts:
- added G***: LOGO, Airbus:Airbus, F.Cu at (320.2, 179.8)
- renumbered X44_b1 to X44_Buzzer1, X44__y1 to X44__Gelb1, X44__g1 to X44__Grün1, X44__r1 to X44__Rot1
Connections:
- REF** pad 1: (no net) -> GND (x22)
- TOOL-FAN0 pad 1: /Fan/X48-FAN0 PIN4 -> /Fan/X48-FAN0 PIN9
- TOOL-FAN0 pad 2: /Fan/X48-FAN0 PIN9 -> /Fan/X48-FAN0 PIN4
Routing:
- net Net-(EndStopZ3-Pin_3): track 284.7 -> 283.5 mm
- net /Fan/X48-FAN0 PIN4: track 176.1 -> 175.1 mm
Other:
- board text added: "DS Airborne Solutions GmbH designed by M. Ick Version 1.0"
