File: kicad/Adapterplatine/temp.kicad_sch (KiCad schematic)
At the start: 12 parts, among them X20 Conn_01x02_Pin, X22 Conn_01x02_Pin, X23 Conn_01x02_Pin, X56 Conn_01x02_Pin

Commit message: Bessere Verlegungen Adapterplatine
Parts:
- removed SPI4: Conn_02x04_Top_Bottom, Connector_PinHeader_2.54mm:PinHeader_2x04_P2.54mm_Vertical, symbol Connector_Generic:Conn_02x04_Top_Bottom
- added SPI4: Conn_02x04_Odd_Even, Connector_PinHeader_2.54mm:PinHeader_2x04_P2.54mm_Vertical, symbol Connector_Generic:Conn_02x04_Odd_Even
Connections:
- net +5V: now also SPI4.1 (Pin_1)
- net GND: now also SPI4.2 (Pin_2), SPI4.8 (Pin_8)
- net at MAX31865_IN1.4 (Pin_4): now also SPI4.4 (Pin_4)
- net at MAX31865_IN1.6 (Pin_6): now also SPI4.6 (Pin_6)
- net at MAX31865_IN1.7 (Pin_7): now also SPI4.3 (Pin_3)
- net at MAX31865_IN1.5 (Pin_5): now also SPI4.5 (Pin_5)
- new net +3.3V: SPI4.7 (Pin_7)

Commit message: Abschlussbericht angefangen/ Adapterplatine ECR DCR
Connections:
- no-connect marks 0 -> 4
Changed lines of the file:
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@@
 	(generator_version "10.0")
 	(paper "A4")
+	(no_connect
+		(at 177.8 71.12)
+	)
+	(no_connect
+		(at 125.73 78.74)
+	)
+	(no_connect
+		(at 125.73 71.12)
+	)
+	(no_connect
+		(at 177.8 83.82)
+	)
 	(wire
 		(pts
@@
 	(wire
 		(pts
+			(xy 179.07 66.04) (xy 177.8 66.04)
+		)
+		(stroke
+			(width 0)
+			(type default)
+		)
+	)
+	(wire
+		(pts
 			(xy 187.96 92.71) (xy 200.66 92.71)
 		)
@@
 	(wire
 		(pts
+			(xy 179.07 68.58) (xy 177.8 68.58)
+		)
+		(stroke
+			(width 0)
+			(type default)
+		)
+	)
+	(wire
+		(pts
+			(xy 198.12 82.55) (xy 198.12 81.28)
+		)
+		(stroke
+			(width 0)
+			(type default)
+		)
+	)
+	(wire
+		(pts
 			(xy 101.6 73.66) (xy 125.73 73.66)
 		)
@@
 	(wire
 		(pts
+			(xy 198.12 67.31) (xy 198.12 68.58)
+		)
+		(stroke
+			(width 0)
+			(type default)
+		)
+	)
+	(wire
+		(pts
+			(xy 205.74 67.31) (xy 205.74 68.58)
+		)
+		(stroke
+			(width 0)
+			(type default)
+		)
+	)
+	(wire
+		(pts
 			(xy 187.96 81.28) (xy 187.96 92.71)
 		)
@@
 		(pts
 			(xy 189.23 76.2) (xy 189.23 90.17)
+		)
+		(stroke
+			(width 0)
+			(type default)
+		)
+	)
+	(wire
+		(pts
+			(xy 205.74 83.82) (xy 205.74 81.28)
 		)
 		(stroke
@@
 	(hierarchical_label "+3.3V"
 		(shape output)
-		(at 205.74 81.28 270)
+		(at 205.74 83.82 270)
 		(effects
 			(font
@@
 	(symbol
 		(lib_id "power:GND")
-		(at 198.12 68.58 180)
+		(at 198.12 67.31 180)
 		(unit 1)
 		(body_style 1)
@@
 		(dnp no)
 		(property "Reference" "#PWR035"
-			(at 198.12 62.23 0)
+			(at 198.12 60.96 0)
 			(hide yes)
 			(show_name no)
@@
 		)
 		(property "Value" "GND"
-			(at 198.12 63.5 90)
+			(at 198.12 62.23 90)
 			(show_name no)
 			(do_not_autoplace no)
@@
 		)
 		(property "Footprint" ""
-			(at 198.12 68.58 0)
+			(at 198.12 67.31 0)
 			(hide yes)
 			(show_name no)
@@
 		)
 		(property "Datasheet" ""
-			(at 198.12 68.58 0)
+			(at 198.12 67.31 0)
 			(hide yes)
 			(show_name no)
@@
 		)
 		(property "Description" "Power symbol creates a global label with name \"GND\" , ground"
-			(at 198.12 68.58 0)
+			(at 198.12 67.31 0)
 			(hide yes)
 			(show_name no)
@@
 	(symbol
 		(lib_id "power:VCC")
-		(at 177.8 66.04 270)
+		(at 179.07 66.04 270)
 		(unit 1)
 		(body_style 1)
@@
 		(dnp no)
 		(property "Reference" "#PWR032"
-			(at 173.99 66.04 0)
+			(at 175.26 66.04 0)
 			(hide yes)
 			(show_name no)
@@
 		)
 		(property "Value" "+5V"
-			(at 182.88 66.04 90)
+			(at 184.15 66.04 90)
 			(show_name no)
 			(do_not_autoplace no)
@@
 		)
 		(property "Footprint" ""
-			(at 177.8 66.04 0)
+			(at 179.07 66.04 0)
 			(hide yes)
 			(show_name no)
@@
 		)
 		(property "Datasheet" ""
-			(at 177.8 66.04 0)
+			(at 179.07 66.04 0)
 			(hide yes)
 			(show_name no)
@@
 		)
 		(property "Description" "Power symbol creates a global label with name \"VCC\""
-			(at 177.8 66.04 0)
+			(at 179.07 66.04 0)
 			(hide yes)
 			(show_name no)
@@
 	(symbol
 		(lib_id "power:GND")
-		(at 205.74 68.58 180)
+		(at 205.74 67.31 180)
 		(unit 1)
 		(body_style 1)
@@
 		(dnp no)
 		(property "Reference" "#PWR037"
-			(at 205.74 62.23 0)
+			(at 205.74 60.96 0)
 			(hide yes)
 			(show_name no)
@@
 		)
 		(property "Value" "GND"
-			(at 205.74 63.5 90)
+			(at 205.74 62.23 90)
 			(show_name no)
 			(do_not_autoplace no)
@@
 		)
 		(property "Footprint" ""
-			(at 205.74 68.58 0)
+			(at 205.74 67.31 0)
 			(hide yes)
 			(show_name no)
@@
 		)
 		(property "Datasheet" ""
-			(at 205.74 68.58 0)
+			(at 205.74 67.31 0)
 			(hide yes)
 			(show_name no)
@@
 		)
 		(property "Description" "Power symbol creates a global label with name \"GND\" , ground"
-			(at 205.74 68.58 0)
+			(at 205.74 67.31 0)
 			(hide yes)
 			(show_name no)
@@
 	(symbol
 		(lib_id "power:GND")
-		(at 177.8 68.58 90)
+		(at 179.07 68.58 90)
 		(unit 1)
 		(body_style 1)
@@
 		(dnp no)
 		(property "Reference" "#PWR024"
-			(at 184.15 68.58 0)
+			(at 185.42 68.58 0)
 			(hide yes)
 			(show_name no)
@@
 		)
 		(property "Value" "GND"
-			(at 182.88 68.58 90)
+			(at 184.15 68.58 90)
 			(show_name no)
 			(do_not_autoplace no)
@@
 		)
 		(property "Footprint" ""
-			(at 177.8 68.58 0)
+			(at 179.07 68.58 0)
 			(hide yes)
 			(show_name no)
@@
 		)
 		(property "Datasheet" ""
-			(at 177.8 68.58 0)
+			(at 179.07 68.58 0)
 			(hide yes)
 			(show_name no)
@@
 		)
 		(property "Description" "Power symbol creates a global label with name \"GND\" , ground"
-			(at 177.8 68.58 0)
+			(at 179.07 68.58 0)
 			(hide yes)
 			(show_name no)
@@
 	(symbol
 		(lib_id "power:VCC")
-		(at 198.12 81.28 180)
+		(at 198.12 82.55 180)
 		(unit 1)
 		(body_style 1)
@@
 		(dnp no)
 		(property "Reference" "#PWR041"
-			(at 198.12 77.47 0)
+			(at 198.12 78.74 0)
 			(hide yes)
 			(show_name no)
@@
 		)
 		(property "Value" "+5V"
-			(at 198.12 86.36 90)
+			(at 198.12 87.63 90)
 			(show_name no)
 			(do_not_autoplace no)
@@
 		)
 		(property "Footprint" ""
-			(at 198.12 81.28 0)
+			(at 198.12 82.55 0)
 			(hide yes)
 			(show_name no)
@@
 		)
 		(property "Datasheet" ""
-			(at 198.12 81.28 0)
+			(at 198.12 82.55 0)
 			(hide yes)
 			(show_name no)
@@
 		)
 		(property "Description" "Power symbol creates a global label with name \"VCC\""
-			(at 198.12 81.28 0)
-			(hide yes)
-			(show_name no)
+			(at 198.12 82.55 0)
+			(hide yes)
+			(show_name no)

Commit message: Adapterplatine Version 1.0
Parts:
- removed MAX31865_OUT1: Conn_01x04_Pin, TerminalBlock_Phoenix:TerminalBlock_Phoenix_PT-1,5-4-3.5-H_1x04_P3.50mm_Horizontal, symbol Connector_Generic:Conn_01x04
- added MAX31865_OUT1, MAX31865_OUT2, MAX31865_OUT3, MAX31865_OUT4: Conn_01x01, Connector_PinSocket_2.54mm:PinSocket_1x01_P2.54mm_Vertical, symbol Connector_Generic:Conn_01x01
Connections:
- net at X22.1 (Pin_1): now also MAX31865_OUT2.1 (Pin_1)
- net at X22.2 (Pin_2): now also MAX31865_OUT3.1 (Pin_1)
Other:
- moved on the sheet: X22
