File: kicad/Adapterplatine/raspi.kicad_sch (KiCad schematic)
At the start: 16 parts, among them X30 Conn_01x05_Pin, X31 Conn_01x05_Pin, X43 Conn_01x05_Pin

Commit message: Adapterplatine Version 1.0 final
Parts:
- added RP2040-PIN9-13: Conn_01x05, Connector_PinSocket_2.54mm:PinSocket_1x05_P2.54mm_Vertical, symbol Connector_Generic:Conn_01x05
- Rasp1: footprint Connector_PinHeader_2.54mm:PinHeader_2x20_P2.54mm_Vertical -> Connector_IDC:IDC-Header_2x20_P2.54mm_Vertical
Connections:
- net +5 VCC: now also Rasp1.2 (Pin_2); no longer Rasp1.1 (Pin_1)
- net GND: now also Rasp1.12 (Pin_12), Rasp1.20 (Pin_20), Rasp1.25 (Pin_25), Rasp1.30 (Pin_30), Rasp1.34 (Pin_34), Rasp1.39 (Pin_39), Rasp1.6 (Pin_6), Rasp1.9 (Pin_9); no longer Rasp1.10 (Pin_10), Rasp1.11 (Pin_11), Rasp1.19 (Pin_19), Rasp1.26 (Pin_26), Rasp1.29 (Pin_29), Rasp1.33 (Pin_33), Rasp1.40 (Pin_40), Rasp1.5 (Pin_5)
- net at RP2040-PIN0-8.1 (Pin_1): now also Rasp1.29 (Pin_29); no longer Rasp1.30 (Pin_30)
- net at Rasp1.7 (Pin_7): now also RP2040-PIN0-8.2 (Pin_2); no longer UART0.2 (Pin_2)
- net at Rasp1.8 (Pin_8): now also UART0.2 (Pin_2); no longer RP2040-PIN0-8.2 (Pin_2)
- net at UART0.1 (Pin_1): now also Rasp1.10 (Pin_10); no longer Rasp1.9 (Pin_9)
- no-connect marks 40 -> 45
Other:
- moved on the sheet: Rasp1
Changed lines of the file:
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@@
 	)
 	(no_connect
+		(at 184.15 129.54)
+	)
+	(no_connect
 		(at 125.73 93.98)
 	)
@@
 	)
 	(no_connect
+		(at 181.61 129.54)
+	)
+	(no_connect
 		(at 113.03 124.46)
 	)
@@
 	)
 	(no_connect
+		(at 179.07 129.54)
+	)
+	(no_connect
 		(at 171.45 110.49)
 	)
@@
 	)
 	(no_connect
+		(at 176.53 129.54)
+	)
+	(no_connect
 		(at 113.03 111.76)
 	)
@@
 	)
 	(no_connect
+		(at 186.69 129.54)
+	)
+	(no_connect
 		(at 190.5 120.65)
 	)
@@
 	(wire
 		(pts
-			(xy 135.89 99.06) (xy 135.89 91.44)
+			(xy 135.89 91.44) (xy 135.89 99.06)
+		)
+		(stroke
+			(width 0)
+			(type default)
+		)
+	)
+	(wire
+		(pts
+			(xy 135.89 100.33) (xy 135.89 119.38)
 		)
 		(stroke
@@
 	(wire
 		(pts
-			(xy 135.89 100.33) (xy 135.89 119.38)
-		)
-		(stroke
-			(width 0)
-			(type default)
-		)
-	)
-	(wire
-		(pts
 			(xy 189.23 66.04) (xy 187.96 66.04)
 		)
@@
 	(wire
 		(pts
+			(xy 113.03 91.44) (xy 110.49 91.44)
+		)
+		(stroke
+			(width 0)
+			(type default)
+		)
+	)
+	(wire
+		(pts
 			(xy 113.03 114.3) (xy 110.49 114.3)
 		)
@@
 		)
 	)
-	(wire
-		(pts
-			(xy 113.03 91.44) (xy 110.49 91.44)
-		)
-		(stroke
-			(width 0)
-			(type default)
-		)
-	)
 	(label "+5 VCC"
 		(at 137.16 128.27 0)
@@
 	(symbol
 		(lib_id "Connector_Generic:Conn_02x20_Odd_Even")
-		(at 118.11 104.14 0)
-		(mirror x)
+		(at 120.65 104.14 180)
 		(unit 1)
 		(body_style 1)
@@
 		(dnp no)
 		(property "Reference" "Rasp1"
-			(at 119.634 74.93 0)
+			(at 119.126 74.93 0)
 			(show_name no)
 			(do_not_autoplace no)
@@
 		)
 		(property "Value" "Conn_02x20_Pin"
-			(at 117.348 72.39 0)
+			(at 121.412 72.39 0)
 			(show_name no)
 			(do_not_autoplace no)
@@
 			)
 		)
-		(property "Footprint" "Connector_PinHeader_2.54mm:PinHeader_2x20_P2.54mm_Vertical"
-			(at 118.11 104.14 0)
+		(property "Footprint" "Connector_IDC:IDC-Header_2x20_P2.54mm_Vertical"
+			(at 120.65 104.14 0)
 			(hide yes)
 			(show_name no)
@@
 		)
 		(property "Datasheet" ""
-			(at 118.11 104.14 0)
+			(at 120.65 104.14 0)
 			(hide yes)
 			(show_name no)
@@
 		)
 		(property "Description" "Generic connector, double row, 02x20, odd/even pin numbering scheme (row 1 odd numbers, row 2 even numbers), script generated (kicad-library-utils/schlib/autogen/connector/)"
-			(at 118.11 104.14 0)
+			(at 120.65 104.14 0)
 			(hide yes)
 			(show_name no)
@@
 		)
 		(property "Hersteller" ""
-			(at 118.11 104.14 0)
+			(at 120.65 104.14 0)
 			(hide yes)
 			(show_name no)
@@
 		)
 		(property "Herstellerbezeichnung" ""
-			(at 118.11 104.14 0)
+			(at 120.65 104.14 0)
 			(hide yes)
 			(show_name no)
@@
 		)
 		(property "Alternative" ""
-			(at 118.11 104.14 0)
+			(at 120.65 104.14 0)
 			(hide yes)
 			(show_name no)
@@
 					(unit 1)
 				)
+			)
+		)
+	)
+	(symbol
+		(lib_id "Connector_Generic:Conn_01x05")
+		(at 181.61 134.62 270)
+		(unit 1)
+		(body_style 1)
+		(exclude_from_sim no)
+		(in_bom yes)
+		(on_board yes)
+		(in_pos_files yes)
+		(dnp no)
+		(fields_autoplaced yes)
+		(property "Reference" "RP2040-PIN9-13"
+			(at 181.61 138.43 90)
+			(show_name no)
+			(do_not_autoplace no)
+			(effects
+				(font
+					(size 1.27 1.27)
+				)
+			)
+		)
+		(property "Value" "Conn_01x05"
+			(at 181.61 140.97 90)
+			(show_name no)
+			(do_not_autoplace no)
+			(effects
+				(font
+					(size 1.27 1.27)
+				)
+			)
+		)
+		(property "Footprint" "Connector_PinSocket_2.54mm:PinSocket_1x05_P2.54mm_Vertical"
+			(at 181.61 134.62 0)
+			(hide yes)
+			(show_name no)
+			(do_not_autoplace no)
+			(effects
+				(font
+					(size 1.27 1.27)
+				)
+			)
+		)
+		(property "Datasheet" ""
+			(at 181.61 134.62 0)
+			(hide yes)
+			(show_name no)
+			(do_not_autoplace no)
+			(effects
+				(font
+					(size 1.27 1.27)
+				)
+			)
+		)
+		(property "Description" "Generic connector, single row, 01x05, script generated (kicad-library-utils/schlib/autogen/connector/)"
+			(at 181.61 134.62 0)
+			(hide yes)
+			(show_name no)
+			(do_not_autoplace no)
+			(effects
+				(font
+					(size 1.27 1.27)
+				)
+			)
+		)
+		(property "Hersteller" ""
+			(at 181.61 134.62 0)
+			(hide yes)
+			(show_name no)
+			(do_not_autoplace no)
+			(effects
+				(font
+					(size 1.27 1.27)
+				)
+			)
+		)
+		(property "Herstellerbezeichnung" ""
+			(at 181.61 134.62 0)
+			(hide yes)
+			(show_name no)
+			(do_not_autoplace no)
+			(effects
+				(font
+					(size 1.27 1.27)
+				)
+			)
+		)
+		(property "Alternative" ""
+			(at 181.61 134.62 0)
+			(hide yes)
+			(show_name no)
+			(do_not_autoplace no)
+			(effects
+				(font
+					(size 1.27 1.27)
+				)
+			)
+		)
+		(pin "5"
+		)
+		(pin "4"
+		)
+		(pin "1"
+		)
+		(pin "3"
+		)
+		(pin "2"
+		)
+		(instances
+			(project "Adapterplatine"
+				(path "/99d5d967-6a35-454f-aac3-01cafa1d30b4/6e4113d7-0438-4c79-b883-7b55fbeab670"
+					(reference "RP2040-PIN9-13")
+					(unit 1)
+				)
