File: kicad/Adapterplatine v1.1/Adapterplatine.kicad_pcb (KiCad board)
At the start: 4 copper layers, 333 x 210 mm, 119 parts, among them J2 Conn_01x05_Pin, J3 Conn_01x04_Pin, J4 Conn_01x03_Pin, X1 Conn_01x02_Pin, X10 Conn_01x04_Pin, X12 Conn_01x05_Pin, X13 Conn_01x05_Pin, X15 Conn_01x05_Pin, X16 Conn_01x05_Pin, X20 Conn_01x02_Pin, X22 Conn_01x02_Pin, X23 Conn_01x02_Pin, X25_1 Conn_01x02_Pin, X28_1 Conn_01x05_Pin, X29_1 Conn_01x05_Pin, X3 Conn_01x02_Pin, X30 Conn_01x05_Pin, X31 Conn_01x05_Pin, X36A1 DE9_Pins, X36B1 DE9_Socket, X37 Conn_01x02_Pin, X38 Conn_01x02_Pin, X39 Conn_01x02_Pin, X40 Conn_01x02_Pin, X43 Conn_01x05_Pin, X44 Conn_01x05_Pin, X44_B1 Conn_01x02_Pin, X44_G1 Conn_01x04_Pin, X44_R1 Conn_01x04_Pin, X44_Y1 Conn_01x02_Pin, X45 DE9_Pins, X46 Conn_02x05_Odd_Even, X48 Conn_02x10_Top_Bottom, X5 Conn_01x04_Pin, X52 Conn_01x05_Pin, X56 Conn_01x02_Pin, X6 Conn_01x04_Pin, X7 Conn_01x04_Pin, X9 Conn_01x04_Pin

Commit message: Kleine Änderungen
Routing:
- net Net-(MAX31865_IN1-Pin_6): track 77.5 -> 80.3 mm
- net Net-(X31-Pin_2): track 28.1 -> 29.8 mm
- net Net-(X30-Pin_2): track 33.6 -> 34.8 mm
- net Net-(X30-Pin_3): track 25.2 -> 26.4 mm
- net Net-(MAX31865_IN1-Pin_7): track 69.6 -> 68.7 mm
Changed lines of the file:
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@@
 	)
 	(image
-		(at 613.669584 125.471806)
+		(at 614.949584 125.471806)
 		(layer "Edge.Cuts")
 		(data "/9j/4AAQSkZJRgABAgEAkACQAAD/2wBDAAEBAQEBAQEBAQEBAQEBAQEBAQEBAQEBAQEBAQEBAQEB"
@@
 	)
 	(image
-		(at 192.551334 125.250001)
+		(at 663.180001 127.020001)
 		(layer "Edge.Cuts")
 		(data "iVBORw0KGgoAAAANSUhEUgAAD3AAAAmOCAIAAABgeqpgAAAAA3NCSVQICAjb4U/gAAAACXBIWXMA"
@@
 	)
 	(image
-		(at 787.169583 125.996111)
+		(at 788.449583 125.996111)
 		(layer "Edge.Cuts")
 		(data "/9j/4AAQSkZJRgABAgEAkACQAAD/2wBDAAEBAQEBAQEBAQEBAQEBAQEBAQEBAQEBAQEBAQEBAQEB"
@@
 	)
 	(segment
-		(start 26.7 44.83)
-		(end 31.87 50)
+		(start 28.04 28.46)
+		(end 26.7 29.8)
+		(width 0.5)
+		(layer "F.Cu")
+		(net "Net-(X30-Pin_3)")
+	)
+	(segment
+		(start 29 28.46)
+		(end 28.04 28.46)
 		(width 0.5)
 		(layer "F.Cu")
@@
 	(segment
 		(start 26.7 29.8)
-		(end 26.7 44.83)
+		(end 26.7 46.8)
 		(width 0.5)
 		(layer "F.Cu")
@@
 	)
 	(segment
-		(start 29 28.46)
-		(end 28.04 28.46)
+		(start 26.7 46.8)
+		(end 29.9 50)
 		(width 0.5)
 		(layer "F.Cu")
@@
 	)
 	(segment
-		(start 28.04 28.46)
-		(end 26.7 29.8)
+		(start 29.9 50)
+		(end 31.87 50)
 		(width 0.5)
 		(layer "F.Cu")
@@
 	)
 	(segment
-		(start 27.88 25.92)
-		(end 25.8 28)
+		(start 29.83 55)
+		(end 31.87 55)
 		(width 0.5)
 		(layer "F.Cu")
@@
 	)
 	(segment
-		(start 25.8 48.93)
-		(end 31.87 55)
+		(start 27.88 25.92)
+		(end 25.8 28)
 		(width 0.5)
 		(layer "F.Cu")
@@
 	)
 	(segment
+		(start 25.8 50.97)
+		(end 29.83 55)
+		(width 0.5)
+		(layer "F.Cu")
+		(net "Net-(X30-Pin_2)")
+	)
+	(segment
 		(start 25.8 28)
-		(end 25.8 48.93)
+		(end 25.8 50.97)
 		(width 0.5)
 		(layer "F.Cu")
@@
 	)
 	(segment
+		(start 163.6 32.4)
+		(end 163.6 30.5)
+		(width 1)
+		(layer "F.Cu")
+		(net "/Motor Driver/X48-Servo-PIN9")
+	)
+	(segment
 		(start 159.6 36.4)
 		(end 163.6 32.4)
@@
 	)
 	(segment
-		(start 163.6 32.4)
-		(end 163.6 30.5)
+		(start 137.33 36.4)
+		(end 159.6 36.4)
 		(width 1)
 		(layer "F.Cu")
@@
 		(net "/Motor Driver/X48-Servo-PIN9")
 	)
-	(segment
-		(start 134.8 36.4)
-		(end 159.6 36.4)
-		(width 1)
-		(layer "F.Cu")
-		(net "/Motor Driver/X48-Servo-PIN9")
-	)
 	(via
-		(at 134.8 36.4)
+		(at 137.33 36.4)
 		(size 1.2)
 		(drill 0.6)
@@
 	)
 	(segment
-		(start 77.9 42)
+		(start 132.49 34.7)
 		(end 85.2 34.7)
 		(width 1)
@@
 	)
 	(segment
-		(start 77.9 59.5)
-		(end 77.9 42)
+		(start 137.33 36.4)
+		(end 134.19 36.4)
 		(width 1)
 		(layer "In1.Cu")
@@
 	)
 	(segment
-		(start 132.4 36.4)
-		(end 134.8 36.4)
+		(start 85.2 34.7)
+		(end 77.9 42)
 		(width 1)
 		(layer "In1.Cu")
@@
 	)
 	(segment
-		(start 130.7 34.7)
-		(end 132.4 36.4)
+		(start 77.9 42)
+		(end 77.9 59.5)
 		(width 1)
 		(layer "In1.Cu")
@@
 	)
 	(segment
-		(start 85.2 34.7)
-		(end 130.7 34.7)
+		(start 134.19 36.4)
+		(end 132.49 34.7)
 		(width 1)
 		(layer "In1.Cu")
@@
 	(segment
 		(start 296.5 152)
-		(end 320 152)
+		(end 322.04 152)
+		(width 0.5)
+		(layer "F.Cu")
+		(net "Net-(MAX31865_IN1-Pin_5)")
+	)
+	(segment
+		(start 322.04 152)
+		(end 333.12 140.92)
 		(width 0.5)
 		(layer "F.Cu")
@@
 	)
 	(segment
-		(start 331.08 140.92)
+		(start 333.12 140.92)
 		(end 337.25 140.92)
 		(width 0.5)
@@
 	)
 	(segment
-		(start 320 152)
-		(end 331.08 140.92)
+		(start 295.97 159.33)
+		(end 300 155.3)
 		(width 0.5)
 		(layer "F.Cu")
-		(net "Net-(MAX31865_IN1-Pin_5)")
+		(net "Net-(MAX31865_IN1-Pin_6)")
 	)
 	(segment
-		(start 286.93 156.57)
-		(end 286.93 158.23)
+		(start 286.9 159.33)
+		(end 295.97 159.33)
 		(width 0.5)
 		(layer "F.Cu")
@@
 	)
 	(segment
-		(start 338.2 155.3)
-		(end 340 153.5)
+		(start 287.09 154.51)
+		(end 285.927 155.673)
 		(width 0.5)
 		(layer "F.Cu")
@@
 	)
 	(segment
-		(start 287.8 159.1)
-		(end 296.2 159.1)
+		(start 340 153.5)
+		(end 340 139.5)
 		(width 0.5)
 		(layer "F.Cu")
@@
 	)
 	(segment
-		(start 296.2 159.1)
-		(end 300 155.3)
+		(start 338.2 155.3)
+		(end 340 153.5)
 		(width 0.5)
 		(layer "F.Cu")
@@
 	)
 	(segment
-		(start 338.88 138.38)
-		(end 337.25 138.38)
+		(start 340 139.5)
+		(end 338.88 138.38)
 		(width 0.5)
 		(layer "F.Cu")
@@
 	)
 	(segment
-		(start 340 139.5)
-		(end 338.88 138.38)
+		(start 285.927 158.357)
+		(end 286.9 159.33)
 		(width 0.5)
 		(layer "F.Cu")
@@
 	(segment
 		(start 288.99 154.51)
-		(end 286.93 156.57)
+		(end 287.09 154.51)
 		(width 0.5)
 		(layer "F.Cu")
@@
 	)
 	(segment
-		(start 286.93 158.23)
-		(end 287.8 159.1)
+		(start 338.88 138.38)
+		(end 337.25 138.38)
 		(width 0.5)
 		(layer "F.Cu")
@@
 	)
 	(segment
-		(start 340 153.5)
-		(end 340 139.5)
+		(start 285.927 155.673)
+		(end 285.927 158.357)
 		(width 0.5)
 		(layer "F.Cu")
@@
 	)
 	(segment
-		(start 286 151)
-		(end 286.97 151.97)
+		(start 337.25 135.84)
+		(end 333.84 135.84)
 		(width 0.5)
 		(layer "F.Cu")
@@
 	)
 	(segment
-		(start 337.25 135.84)
-		(end 333.84 135.84)
+		(start 286.97 151.97)
+		(end 288.99 151.97)
 		(width 0.5)
 		(layer "F.Cu")
@@
 	)
 	(segment
-		(start 333.84 135.84)
-		(end 331.5 133.5)
+		(start 286 151)
+		(end 286.97 151.97)
 		(width 0.5)
 		(layer "F.Cu")
@@
 	)
 	(segment
-		(start 292 133.5)
-		(end 286 139.5)
+		(start 333.84 135.84)
+		(end 332.61 134.61)
 		(width 0.5)
 		(layer "F.Cu")
@@
 	)
 	(segment
-		(start 286.97 151.97)
-		(end 288.99 151.97)
+		(start 290.89 134.61)
+		(end 286 139.5)
 		(width 0.5)
 		(layer "F.Cu")
@@
 	)
 	(segment
-		(start 331.5 133.5)
-		(end 292 133.5)
+		(start 332.61 134.61)
+		(end 290.89 134.61)
 		(width 0.5)
 		(layer "F.Cu")
@@
 	)
 	(segment
-		(start 29 39.1)
-		(end 29 43.015)
+		(start 42.1 26)
+		(end 27.8 40.3)
 		(width 0.5)
 		(layer "F.Cu")
@@
 	)
 	(segment
-		(start 29 43.015)
-		(end 30.935 44.95)
+		(start 27.8 43.01)
+		(end 29.74 44.95)
 		(width 0.5)
 		(layer "F.Cu")
@@
 	)
 	(segment
-		(start 30.935 44.95)
-		(end 31.92 44.95)
+		(start 27.8 40.3)
+		(end 27.8 43.01)
 		(width 0.5)
 		(layer "F.Cu")
@@
 	)
 	(segment
-		(start 42.1 26)
-		(end 29 39.1)
+		(start 29.74 44.95)
+		(end 31.92 44.95)
 		(width 0.5)
 		(layer "F.Cu")
