File: kicad/Adapterplatine v1.1/Adapterplatine.kicad_pcb (KiCad board)
At the start: 4 copper layers, 333 x 210 mm, 119 parts, among them J2 Conn_01x05_Pin, J3 Conn_01x04_Pin, J4 Conn_01x03_Pin, X1 Conn_01x02_Pin, X10 Conn_01x04_Pin, X12 Conn_01x05_Pin, X13 Conn_01x05_Pin, X15 Conn_01x05_Pin, X16 Conn_01x05_Pin, X20 Conn_01x02_Pin, X22 Conn_01x02_Pin, X23 Conn_01x02_Pin, X25_1 Conn_01x02_Pin, X28_1 Conn_01x05_Pin, X29_1 Conn_01x05_Pin, X3 Conn_01x02_Pin, X30 Conn_01x05_Pin, X31 Conn_01x05_Pin, X36A1 DE9_Pins, X36B1 DE9_Socket, X37 Conn_01x02_Pin, X38 Conn_01x02_Pin, X39 Conn_01x02_Pin, X40 Conn_01x02_Pin, X43 Conn_01x05_Pin, X44 Conn_01x05_Pin, X44_B1 Conn_01x02_Pin, X44_G1 Conn_01x04_Pin, X44_R1 Conn_01x04_Pin, X44_Y1 Conn_01x02_Pin, X45 DE9_Pins, X46 Conn_02x05_Odd_Even, X48 Conn_02x10_Top_Bottom, X5 Conn_01x04_Pin, X52 Conn_01x05_Pin, X56 Conn_01x02_Pin, X6 Conn_01x04_Pin, X7 Conn_01x04_Pin, X9 Conn_01x04_Pin

Commit message: Ansatz F421 im Finalen Bericht/ Einbindung Flowsensoren I²C/ DFX Dateien KiCad wieder F.Fab
Parts:
- moved X29_1 12.0 mm to (55.5, 226.0)
- moved R3 4.52 mm to (33.9, 220.5)
- moved X15 4.52 mm to (34.0, 226.0)
- moved J4 3.00 mm to (161.6, 210.5)
- moved J3 2.00 mm to (161.5, 218.0)
Routing:
- net Net-(I2C1-Pin_3): track 457.0 -> 451.5 mm
- net Net-(I2C1-Pin_4): track 452.1 -> 447.1 mm
- net /Platines/+3.3V: track 524.3 -> 520.7 mm
- net Net-(ChamberFAN1-Pin_1): track 154.3 -> 151.9 mm
- net Net-(EndStopZ3-Pin_3): track 283.5 -> 281.6 mm
- net /Fan/Blower_PG: track 173.7 -> 173.1 mm
- net /Fan/Blower_PWM: track 187.7 -> 187.2 mm
