File: kicad/Adapterplatine v1.1/Adapterplatine.kicad_pcb (KiCad board)
At the start: 4 copper layers, 333 x 210 mm, 122 parts, among them J2 Conn_01x05_Pin, J3 Conn_01x04_Pin, J4 Conn_01x03_Pin, X1 Conn_01x02_Pin, X10 Conn_01x04_Pin, X12 Conn_01x05_Pin, X13 Conn_01x05_Pin, X15 Conn_01x05_Pin, X16 Conn_01x05_Pin, X20 Conn_01x02_Pin, X22 Conn_01x02_Pin, X23 Conn_01x02_Pin, X25_1 Conn_01x02_Pin, X28_1 Conn_01x05_Pin, X29_1 Conn_01x05_Pin, X3 Conn_01x02_Pin, X30 Conn_01x05_Pin, X31 Conn_01x05_Pin, X36A1 DE9_Pins, X36B1 DE9_Socket, X37 Conn_01x02_Pin, X38 Conn_01x02_Pin, X39 Conn_01x02_Pin, X40 Conn_01x02_Pin, X43 Conn_01x05_Pin, X44 Conn_01x05_Pin, X44_B1 Conn_01x02_Pin, X44_G1 Conn_01x04_Pin, X44_R1 Conn_01x04_Pin, X44_Y1 Conn_01x02_Pin, X45 DE9_Pins, X46 Conn_02x05_Odd_Even, X48 Conn_02x10_Top_Bottom, X5 Conn_01x04_Pin, X52 Conn_01x05_Pin, X56 Conn_01x02_Pin, X6 Conn_01x04_Pin, X7 Conn_01x04_Pin, X9 Conn_01x04_Pin

Commit message: printer.cfg Anpassungen/ Servo Fehler Platine/KLipper Screen
Connections:
- MAX31865_IN1 pad 1: +5V -> /Platines/+3.3V
- Servo1 pad 1: /Motor Driver/X48-Servo-PIN9 -> /Motor Driver/X48-Servo-PIN10
- Servo1 pad 3: /Motor Driver/X48-Servo-PIN10 -> /Motor Driver/X48-Servo-PIN9
Routing:
- net /Platines/+3.3V: track 518.4 -> 573.9 mm
- net /Motor Driver/X48-Servo-PIN10: track 236.7 -> 243.8 mm
- net /Motor Driver/X48-Servo-PIN9: track 238.9 -> 232.9 mm
- net Net-(MAX31865_IN1-Pin_6): track 80.3 -> 81.9 mm
