File: kicad/Adapterplatine v1.1/platines.kicad_sch (KiCad schematic)
At the start: 6 parts, among them X28_1 Conn_01x05_Pin, X29_1 Conn_01x05_Pin, X46 Conn_02x05_Odd_Even, X48 Conn_02x10_Top_Bottom

Commit message: Platine V1.1 Einbau I2C Heatend Loadcells
Connections:
- net +3.3V: now also X28_1.4 (Pin_4), X48.13 (Pin_13), X48.15 (Pin_15)
- net GND: now also X28_1.1 (Pin_1), X28_1.5 (Pin_5)
- net at I2C1.4 (Pin_4), X29_1.3 (Pin_3): now also X28_1.3 (Pin_3)
- net at I2C1.3 (Pin_3), X29_1.4 (Pin_4): now also X28_1.2 (Pin_2)
- no-connect marks 17 -> 10
Other:
- moved on the sheet: I2C1, X28_1

Commit message: Fehlerbeseitung Adapterplatine
Parts:
- X48: footprint Connector_Molex:Molex_Mini-Fit_Jr_5566-20A_2x10_P4.20mm_Vertical -> Connector_Molex:Molex_Micro-Fit_3.0_43045-2012_2x10_P3.00mm_Vertical
Changed lines of the file:
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@@
 			)
 		)
-		(property "Footprint" "Connector_Molex:Molex_Mini-Fit_Jr_5566-20A_2x10_P4.20mm_Vertical"
+		(property "Footprint" "Connector_Molex:Molex_Micro-Fit_3.0_43045-2012_2x10_P3.00mm_Vertical"
 			(at 199.39 95.25 0)
 			(hide yes)
