File: kicad/Adapterplatine v1.1/motordriver.kicad_sch (KiCad schematic)
At the start: 11 parts, among them X10 Conn_01x04_Pin, X5 Conn_01x04_Pin, X6 Conn_01x04_Pin, X7 Conn_01x04_Pin, X9 Conn_01x04_Pin

Commit message: printer.cfg Anpassungen/ Servo Fehler Platine/KLipper Screen
Connections:
- net X48-Servo-PIN10: now also Servo1.1 (Pin_1); no longer Servo1.3 (Pin_3)
- net X48-Servo-PIN9: now also Servo1.3 (Pin_3); no longer Servo1.1 (Pin_1)
Changed lines of the file:
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@@
+	(wire
+		(pts
+			(xy 210.82 105.41) (xy 210.82 123.19)
+		)
+		(stroke
+			(width 0)
+			(type default)
+		)
+	)
 	(wire
 		(pts
@@
 	(wire
 		(pts
+			(xy 215.9 105.41) (xy 215.9 123.19)
+		)
+		(stroke
+			(width 0)
+			(type default)
+		)
+	)
+	(wire
+		(pts
 			(xy 179.07 110.49) (xy 179.07 118.11)
 		)
@@
 	(wire
 		(pts
-			(xy 215.9 105.41) (xy 215.9 123.19)
-		)
-		(stroke
-			(width 0)
-			(type default)
-		)
-	)
-	(wire
-		(pts
 			(xy 193.04 105.41) (xy 193.04 118.11)
 		)
@@
 		(pts
 			(xy 92.71 110.49) (xy 92.71 118.11)
-		)
-		(stroke
-			(width 0)
-			(type default)
-		)
-	)
-	(wire
-		(pts
-			(xy 210.82 105.41) (xy 210.82 123.19)
 		)
 		(stroke
@@
 	(hierarchical_label "X48-Servo-PIN10"
 		(shape input)
-		(at 215.9 123.19 270)
+		(at 210.82 123.19 270)
 		(effects
 			(font
@@
 	(hierarchical_label "X48-Servo-PIN9"
 		(shape input)
-		(at 210.82 123.19 270)
+		(at 215.9 123.19 270)
 		(effects
 			(font
