File: kicad/Adapterplatine v1.1/temp.kicad_sch (KiCad schematic)
At the start: 15 parts, among them X20 Conn_01x02_Pin, X22 Conn_01x02_Pin, X23 Conn_01x02_Pin, X56 Conn_01x02_Pin

Commit message: Platine V1.1 Einbau I2C Heatend Loadcells
Connections:
- net at SPI4.5 (Pin_5): now also MAX31865_IN1.6 (Pin_6); no longer MAX31865_IN1.5 (Pin_5)
- net at SPI4.6 (Pin_6): now also MAX31865_IN1.5 (Pin_5); no longer MAX31865_IN1.6 (Pin_6)
Changed lines of the file:
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@@
 	(wire
 		(pts
-			(xy 177.8 78.74) (xy 187.96 78.74)
-		)
-		(stroke
-			(width 0)
-			(type default)
-		)
-	)
-	(wire
-		(pts
-			(xy 177.8 76.2) (xy 189.23 76.2)
+			(xy 177.8 76.2) (xy 191.77 76.2)
 		)
 		(stroke
@@
 	(wire
 		(pts
-			(xy 187.96 92.71) (xy 200.66 92.71)
+			(xy 189.23 91.44) (xy 200.66 91.44)
 		)
 		(stroke
@@
 	(wire
 		(pts
-			(xy 203.2 81.28) (xy 203.2 90.17)
-		)
-		(stroke
-			(width 0)
-			(type default)
-		)
-	)
-	(wire
-		(pts
-			(xy 177.8 81.28) (xy 187.96 81.28)
-		)
-		(stroke
-			(width 0)
-			(type default)
-		)
-	)
-	(wire
-		(pts
-			(xy 189.23 90.17) (xy 203.2 90.17)
+			(xy 203.2 81.28) (xy 203.2 92.71)
+		)
+		(stroke
+			(width 0)
+			(type default)
+		)
+	)
+	(wire
+		(pts
+			(xy 177.8 81.28) (xy 189.23 81.28)
+		)
+		(stroke
+			(width 0)
+			(type default)
+		)
+	)
+	(wire
+		(pts
+			(xy 191.77 92.71) (xy 203.2 92.71)
 		)
 		(stroke
@@
 	(wire
 		(pts
+			(xy 191.77 58.42) (xy 191.77 76.2)
+		)
+		(stroke
+			(width 0)
+			(type default)
+		)
+	)
+	(wire
+		(pts
+			(xy 177.8 78.74) (xy 191.77 78.74)
+		)
+		(stroke
+			(width 0)
+			(type default)
+		)
+	)
+	(wire
+		(pts
+			(xy 191.77 92.71) (xy 191.77 78.74)
+		)
+		(stroke
+			(width 0)
+			(type default)
+		)
+	)
+	(wire
+		(pts
 			(xy 111.76 72.39) (xy 111.76 73.66)
 		)
@@
 	(wire
 		(pts
-			(xy 187.96 81.28) (xy 187.96 92.71)
+			(xy 189.23 81.28) (xy 189.23 91.44)
 		)
 		(stroke
@@
 	(wire
 		(pts
-			(xy 187.96 78.74) (xy 187.96 58.42)
-		)
-		(stroke
-			(width 0)
-			(type default)
-		)
-	)
-	(wire
-		(pts
 			(xy 97.79 88.9) (xy 125.73 88.9)
 		)
@@
 	(wire
 		(pts
-			(xy 187.96 58.42) (xy 203.2 58.42)
-		)
-		(stroke
-			(width 0)
-			(type default)
-		)
-	)
-	(wire
-		(pts
-			(xy 200.66 81.28) (xy 200.66 92.71)
+			(xy 191.77 58.42) (xy 203.2 58.42)
+		)
+		(stroke
+			(width 0)
+			(type default)
+		)
+	)
+	(wire
+		(pts
+			(xy 200.66 81.28) (xy 200.66 91.44)
 		)
 		(stroke
@@
 		)
 		(stroke
-			(width 0)
-			(type default)
-		)
-	)
-	(wire
-		(pts
-			(xy 189.23 76.2) (xy 189.23 90.17)
-		)
-		(stroke

Commit message: printer.cfg Anpassungen/ Servo Fehler Platine/KLipper Screen
Connections:
- net +3.3V: now also MAX31865_IN1.1 (Pin_1)
- net +5V: no longer MAX31865_IN1.1 (Pin_1)
Changed lines of the file:
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@@
 	)
 	(hierarchical_label "+3.3V"
-		(shape output)
+		(shape input)
 		(at 205.74 83.82 270)
 		(effects
@@
 			)
 			(justify right)
+		)
+	)
+	(hierarchical_label "+3.3V"
+		(shape input)
+		(at 179.07 66.04 0)
+		(effects
+			(font
+				(size 1.27 1.27)
+			)
+			(justify left)
 		)
 	)
@@
 					(unit 1)
 				)
-			)
-		)
-	)
-	(symbol
-		(lib_id "power:VCC")
-		(at 179.07 66.04 270)
-		(unit 1)
-		(body_style 1)
-		(exclude_from_sim no)
-		(in_bom yes)
-		(on_board yes)
-		(in_pos_files yes)
-		(dnp no)
-		(property "Reference" "#PWR032"
-			(at 175.26 66.04 0)
-			(hide yes)
-			(show_name no)
-			(do_not_autoplace no)
-			(effects
-				(font
-					(size 1.27 1.27)
-				)
-			)
-		)
-		(property "Value" "+5V"
-			(at 184.15 66.04 90)
-			(show_name no)
-			(do_not_autoplace no)
-			(effects
-				(font
-					(size 1.27 1.27)
-				)
-			)
-		)
-		(property "Footprint" ""
-			(at 179.07 66.04 0)
-			(hide yes)
-			(show_name no)
-			(do_not_autoplace no)
-			(effects
-				(font
-					(size 1.27 1.27)
-				)
-			)
-		)
-		(property "Datasheet" ""
-			(at 179.07 66.04 0)
-			(hide yes)
-			(show_name no)
-			(do_not_autoplace no)
-			(effects
-				(font
-					(size 1.27 1.27)
-				)
-			)
-		)
-		(property "Description" "Power symbol creates a global label with name \"VCC\""
-			(at 179.07 66.04 0)
-			(hide yes)
-			(show_name no)
-			(do_not_autoplace no)
-			(effects
-				(font
-					(size 1.27 1.27)
-				)
-			)
-		)
-		(pin "1"
-		)
-		(instances
-			(project "Adapterplatine"
-				(path "/99d5d967-6a35-454f-aac3-01cafa1d30b4/978a6864-b302-4b1a-93ac-77e155af244a"
-					(reference "#PWR032")
-					(unit 1)
-				)
